Commit message: Added the URDF in the .xacro file

File: model/robot.xacro (robot description, xacro)
@@ -156,3 +156,27 @@
     <xacro:inertia_caster/>
   </link>
+  <joint name="lidar_joint" type="fixed">
+    <origin xyz="0 0 ${b+r}" rpy="0 0 0"/>
+    <parent link="body_link"/>
+    <child link="lidar_link"/>
+    <axis xyz="0 1 0" rpy="0 0 0"/>
+  </joint>
+  <link name='lidar_link'>
+    <visual>
+      <origin xyz="0 0 0.5" rpy="0 0 0"/>
+      <geometry>
+        <cylinder length="0.1" radius="0.1"/>
+      </geometry>
+    </visual>
+    <collision>
+      <origin xyz="0 0 0.5" rpy="0 0 0"/>
+      <geometry>
+        <cylinder length="0.1" radius="0.1"/>
+      </geometry>
+    </collision>
+    <inertial>
+      <mass value="1e-6"/>
+      <inertia ixx="1e-6" ixy="0" ixz="0" iyy="1e-6" iyz="0" izz="1e-6"/>
+    </inertial>
+  </link>
 </robot>

Commit message: Funciona el lidar

File: model/robot.xacro (robot description, xacro)
@@ -157,5 +157,5 @@
   </link>
   <joint name="lidar_joint" type="fixed">
-    <origin xyz="0 0 ${b+r}" rpy="0 0 0"/>
+    <origin xyz="0.0 0 ${b+r}" rpy="0 0 0"/>
     <parent link="body_link"/>
     <child link="lidar_link"/>
@@ -164,5 +164,5 @@
   <link name='lidar_link'>
     <visual>
-      <origin xyz="0 0 0.5" rpy="0 0 0"/>
+      <origin xyz="0 0 0.05" rpy="0 0 0"/>
       <geometry>
         <cylinder length="0.1" radius="0.1"/>

Commit message: Modified the position of the lidar_joint

File: model/robot.xacro (robot description, xacro)
@@ -157,5 +157,5 @@
   </link>
   <joint name="lidar_joint" type="fixed">
-    <origin xyz="0.0 0 ${b+r}" rpy="0 0 0"/>
+    <origin xyz="${s3} 0 ${b+r}" rpy="0 0 0"/>
     <parent link="body_link"/>
     <child link="lidar_link"/>

Commit message: Modified the wheel joints orientation

File: model/robot.xacro (robot description, xacro)
@@ -93,6 +93,6 @@
     <parent link="body_link"/>
     <child link="wheel1_link"/>
-    <origin xyz="${-s2} ${-s4} ${r}" rpy="0 0 0"/>
-    <axis xyz="0 1 0"/>
+    <origin xyz="${-s2} ${-s4} ${r}" rpy="${pi_const / 2.0} 0 0"/>
+    <axis xyz="0 0 -1"/>
     <limit effort="50000" velocity="10"/>
     <dynamics damping="1.0" friction="1.0"/>
@@ -100,5 +100,5 @@
   <link name="wheel1_link">
     <visual>
-      <origin rpy="1.570595 0 0" xyz="0 0 0"/>
+      <origin rpy="0 0 0" xyz="0 0 0"/>
       <geometry>
         <cylinder length="${d}" radius="${r}"/>
@@ -106,5 +106,5 @@
     </visual>
     <collision>
-      <origin rpy="1.570595 0 0" xyz="0 0 0"/>
+      <origin rpy="0 0 0" xyz="0 0 0"/>
       <geometry>
         <cylinder length="${d}" radius="${r}"/>
@@ -116,6 +116,6 @@
     <parent link="body_link"/>
     <child link="wheel2_link"/>
-    <origin xyz="${-s2} ${s4} ${r}" rpy="0 0 0"/>
-    <axis xyz="0 1 0"/>
+    <origin xyz="${-s2} ${s4} ${r}" rpy="${-pi_const / 2.0} 0 0"/>
+    <axis xyz="0 0 1"/>
     <limit effort="50000" velocity="10"/>
     <dynamics damping="1.0" friction="1.0"/>
@@ -123,5 +123,5 @@
   <link name="wheel2_link">
     <visual>
-      <origin rpy="1.570595 0 0" xyz="0 0 0"/>
+      <origin rpy="0 0 0" xyz="0 0 0"/>
       <geometry>
         <cylinder length="${d}" radius="${r}"/>
@@ -129,5 +129,5 @@
     </visual>
     <collision>
-      <origin rpy="1.570595 0 0" xyz="0 0 0"/>
+      <origin rpy="0 0 0" xyz="0 0 0"/>
       <geometry>
         <cylinder length="${d}" radius="${r}"/>
@@ -157,12 +157,12 @@
   </link>
   <joint name="lidar_joint" type="fixed">
-    <origin xyz="${s3} 0 ${b+r}" rpy="0 0 0"/>
+    <origin xyz="${s3} 0 ${b+r+0.05}" rpy="0 0 0"/>
     <parent link="body_link"/>
     <child link="lidar_link"/>
-    <axis xyz="0 1 0" rpy="0 0 0"/>
+    <axis xyz="0 0 1" rpy="0 0 0"/>
   </joint>
   <link name='lidar_link'>
     <visual>
-      <origin xyz="0 0 0.05" rpy="0 0 0"/>
+      <origin xyz="0 0 0" rpy="0 0 0"/>
       <geometry>
         <cylinder length="0.1" radius="0.1"/>
@@ -170,5 +170,5 @@
     </visual>
     <collision>
-      <origin xyz="0 0 0.5" rpy="0 0 0"/>
+      <origin xyz="0 0 0" rpy="0 0 0"/>
       <geometry>
         <cylinder length="0.1" radius="0.1"/>

Commit message: Modified the robot dimensions to fit my real prototipe

File: model/robot.xacro (robot description, xacro)
@@ -7,15 +7,15 @@
   <xacro:property name="pi_const" value="3.14159265"/>
   <!-- Body Dimensions -->
-  <xacro:property name="a" value="1"/>
-  <xacro:property name="b" value="0.3"/>
-  <xacro:property name="c" value="0.6"/>
+  <xacro:property name="a" value="0.52"/>
+  <xacro:property name="b" value="0.29"/>
+  <xacro:property name="c" value="0.5"/>
   <!-- Wheel and caster dimensions -->
   <!-- Wheel and caster r -->
-  <xacro:property name="r" value="0.15"/>
+  <xacro:property name="r" value="0.155"/>
   <!-- Wheel height -->
-  <xacro:property name="d" value="0.1"/>
+  <xacro:property name="d" value="0.05"/>
   <xacro:property name="s1" value="${b/2+r}"/>
-  <xacro:property name="s2" value="${2*r}"/>
-  <xacro:property name="s3" value="${2*r}"/>
+  <xacro:property name="s2" value="${(a/2)-r}"/>
+  <xacro:property name="s3" value="${(a/2)-r}"/>
   <xacro:property name="s4" value="${c/2+d/2}"/>
   <!-- ############################################### -->
@@ -27,7 +27,7 @@
   <xacro:property name="d3" value="2710.0"/>
   <!-- Robot body mass, wheel mass, caster mass -->
-  <xacro:property name="m1" value="${d1*a*c*b}"/>
-  <xacro:property name="m2" value="${d2*pi_const*r*r*d}"/>
-  <xacro:property name="m3" value="${d3*(4.0/3.0)*pi_const*r*r*r}"/>
+  <xacro:property name="m1" value="60"/>
+  <xacro:property name="m2" value="1"/>
+  <xacro:property name="m3" value="0.5"/>
   <!-- Moments of inertia of the robot body -->
   <xacro:property name="Ix_body" value="${(1/12)*m1*(b*b+c*c) }" />
@@ -157,5 +157,5 @@
   </link>
   <joint name="lidar_joint" type="fixed">
-    <origin xyz="${s3} 0 ${b+r+0.05}" rpy="0 0 0"/>
+    <origin xyz="0.22 0 ${b+r+0.065}" rpy="0 0 0"/>
     <parent link="body_link"/>
     <child link="lidar_link"/>
@@ -164,13 +164,13 @@
   <link name='lidar_link'>
     <visual>
-      <origin xyz="0 0 0" rpy="0 0 0"/>
+      <origin xyz="0 0 -0.03" rpy="0 0 0"/>
       <geometry>
-        <cylinder length="0.1" radius="0.1"/>
+        <cylinder length="0.08" radius="0.03"/>
       </geometry>
     </visual>
     <collision>
-      <origin xyz="0 0 0" rpy="0 0 0"/>
+      <origin xyz="0 0 -0.03" rpy="0 0 0"/>
       <geometry>
-        <cylinder length="0.1" radius="0.1"/>
+        <cylinder length="0.08" radius="0.03"/>
       </geometry>
     </collision>
